Commit message: Update myrobot.xacro

File: src/robot_description/urdf/myrobot.xacro (robot description, xacro)
@@ -144,5 +144,5 @@
     </inertial>
     <visual>
-        <origin xyz="0.0 0.0 0.1" rpy="0.0 0.0 0.0"/>
+        <origin xyz="0.0 0.0 0.1" rpy="0.0 0.0 1.57"/>
         <geometry>
         <!-- <box size="1.0 1.0 1.0"/> -->
@@ -160,5 +160,5 @@
     <!-- <box size= "1e-10  1e-10 1e-10"/> -->
        <!-- <mesh filename="package://robot_description/meshes/astra.dae"/> -->
-<box size="1.0 1.0 1.0"/>
+<box size="0.1 0.1 0.1"/>
         </geometry>
     </collision>
